Commit message: Move meshes down to per-model subdir.
Also split into visual and collision quality (only visual for now).

File: urdf/Staubli_RX60L.urdf (robot description, URDF)
Before this commit: robot STAUBLI_RX60L, 7 links, 6 joints
Links:
- link Staubli_RX60L_Link1: geometry collision mesh filename=package://staubli/meshes/rx60l/visual/RX60BL_HB.dae scale=0.001 0.001 0.001; visual mesh filename=package://staubli/meshes/rx60l/visual/RX60BL_HB.dae scale=0.001 0.001 0.001
- link Staubli_RX60L_Link2: geometry collision mesh filename=package://staubli/meshes/rx60l/visual/RX60BL_HB1.dae scale=0.001 0.001 0.001; visual mesh filename=package://staubli/meshes/rx60l/visual/RX60BL_HB1.dae scale=0.001 0.001 0.001
- link Staubli_RX60L_Link3: geometry collision mesh filename=package://staubli/meshes/rx60l/visual/RX60BL_HB2.stl scale=0.001 0.001 0.001; visual mesh filename=package://staubli/meshes/rx60l/visual/RX60BL_HB2.stl scale=0.001 0.001 0.001
- link Staubli_RX60L_Link4: geometry collision mesh filename=package://staubli/meshes/rx60l/visual/RX60BL_HB3.dae scale=0.001 0.001 0.001; visual mesh filename=package://staubli/meshes/rx60l/visual/RX60BL_HB3.dae scale=0.001 0.001 0.001
- link Staubli_RX60L_Link5: geometry collision mesh filename=package://staubli/meshes/rx60l/visual/RX60BL_HB4.dae scale=0.001 0.001 0.001; visual mesh filename=package://staubli/meshes/rx60l/visual/RX60BL_HB4.dae scale=0.001 0.001 0.001
- link Staubli_RX60L_Link6: geometry collision mesh filename=package://staubli/meshes/rx60l/visual/RX60BL_HB5.dae scale=0.001 0.001 0.001; visual mesh filename=package://staubli/meshes/rx60l/visual/RX60BL_HB5.dae scale=0.001 0.001 0.001
- link Staubli_RX60L_Link7: geometry collision mesh filename=package://staubli/meshes/rx60l/visual/RX60BL_HB6.dae scale=0.001 0.001 0.001; visual mesh filename=package://staubli/meshes/rx60l/visual/RX60BL_HB6.dae scale=0.001 0.001 0.001

File: urdf/Staubli_RX60L_gripper.urdf (robot description, URDF)
Before this commit: robot STAUBLI_RX60L, 11 links, 10 joints
Links:
- link Staubli_RX60L_Link1: geometry collision mesh filename=package://staubli/meshes/rx60l/visual/RX60BL_HB.dae scale=0.001 0.001 0.001; visual mesh filename=package://staubli/meshes/rx60l/visual/RX60BL_HB.dae scale=0.001 0.001 0.001
- link Staubli_RX60L_Link2: geometry collision mesh filename=package://staubli/meshes/rx60l/visual/RX60BL_HB1.dae scale=0.001 0.001 0.001; visual mesh filename=package://staubli/meshes/rx60l/visual/RX60BL_HB1.dae scale=0.001 0.001 0.001
- link Staubli_RX60L_Link3: geometry collision mesh filename=package://staubli/meshes/rx60l/visual/RX60BL_HB2.stl scale=0.001 0.001 0.001; visual mesh filename=package://staubli/meshes/rx60l/visual/RX60BL_HB2.stl scale=0.001 0.001 0.001
- link Staubli_RX60L_Link4: geometry collision mesh filename=package://staubli/meshes/rx60l/visual/RX60BL_HB3.dae scale=0.001 0.001 0.001; visual mesh filename=package://staubli/meshes/rx60l/visual/RX60BL_HB3.dae scale=0.001 0.001 0.001
- link Staubli_RX60L_Link5: geometry collision mesh filename=package://staubli/meshes/rx60l/visual/RX60BL_HB4.dae scale=0.001 0.001 0.001; visual mesh filename=package://staubli/meshes/rx60l/visual/RX60BL_HB4.dae scale=0.001 0.001 0.001
- link Staubli_RX60L_Link6: geometry collision mesh filename=package://staubli/meshes/rx60l/visual/RX60BL_HB5.dae scale=0.001 0.001 0.001; visual mesh filename=package://staubli/meshes/rx60l/visual/RX60BL_HB5.dae scale=0.001 0.001 0.001
- link Staubli_RX60L_Link7: geometry collision mesh filename=package://staubli/meshes/rx60l/visual/RX60BL_HB6.dae scale=0.001 0.001 0.001; visual mesh filename=package://staubli/meshes/rx60l/visual/RX60BL_HB6.dae scale=0.001 0.001 0.001

Commit message: Convert mesh filenames to lowercase.

File: urdf/Staubli_RX60L.urdf (robot description, URDF)
Before this commit: robot STAUBLI_RX60L, 7 links, 6 joints
Links:
- link Staubli_RX60L_Link1: geometry collision mesh filename=package://staubli/meshes/rx60l/visual/rx60bl_hb.dae scale=0.001 0.001 0.001; visual mesh filename=package://staubli/meshes/rx60l/visual/rx60bl_hb.dae scale=0.001 0.001 0.001
- link Staubli_RX60L_Link2: geometry collision mesh filename=package://staubli/meshes/rx60l/visual/rx60bl_hb1.dae scale=0.001 0.001 0.001; visual mesh filename=package://staubli/meshes/rx60l/visual/rx60bl_hb1.dae scale=0.001 0.001 0.001
- link Staubli_RX60L_Link3: geometry collision mesh filename=package://staubli/meshes/rx60l/visual/rx60bl_hb2.stl scale=0.001 0.001 0.001; visual mesh filename=package://staubli/meshes/rx60l/visual/rx60bl_hb2.stl scale=0.001 0.001 0.001
- link Staubli_RX60L_Link4: geometry collision mesh filename=package://staubli/meshes/rx60l/visual/rx60bl_hb3.dae scale=0.001 0.001 0.001; visual mesh filename=package://staubli/meshes/rx60l/visual/rx60bl_hb3.dae scale=0.001 0.001 0.001
- link Staubli_RX60L_Link5: geometry collision mesh filename=package://staubli/meshes/rx60l/visual/rx60bl_hb4.dae scale=0.001 0.001 0.001; visual mesh filename=package://staubli/meshes/rx60l/visual/rx60bl_hb4.dae scale=0.001 0.001 0.001
- link Staubli_RX60L_Link6: geometry collision mesh filename=package://staubli/meshes/rx60l/visual/rx60bl_hb5.dae scale=0.001 0.001 0.001; visual mesh filename=package://staubli/meshes/rx60l/visual/rx60bl_hb5.dae scale=0.001 0.001 0.001
- link Staubli_RX60L_Link7: geometry collision mesh filename=package://staubli/meshes/rx60l/visual/rx60bl_hb6.dae scale=0.001 0.001 0.001; visual mesh filename=package://staubli/meshes/rx60l/visual/rx60bl_hb6.dae scale=0.001 0.001 0.001

File: urdf/Staubli_RX60L_gripper.urdf (robot description, URDF)
Before this commit: robot STAUBLI_RX60L, 11 links, 10 joints
Links:
- link Staubli_RX60L_Link1: geometry collision mesh filename=package://staubli/meshes/rx60l/visual/rx60bl_hb.dae scale=0.001 0.001 0.001; visual mesh filename=package://staubli/meshes/rx60l/visual/rx60bl_hb.dae scale=0.001 0.001 0.001
- link Staubli_RX60L_Link2: geometry collision mesh filename=package://staubli/meshes/rx60l/visual/rx60bl_hb1.dae scale=0.001 0.001 0.001; visual mesh filename=package://staubli/meshes/rx60l/visual/rx60bl_hb1.dae scale=0.001 0.001 0.001
- link Staubli_RX60L_Link3: geometry collision mesh filename=package://staubli/meshes/rx60l/visual/rx60bl_hb2.stl scale=0.001 0.001 0.001; visual mesh filename=package://staubli/meshes/rx60l/visual/rx60bl_hb2.stl scale=0.001 0.001 0.001
- link Staubli_RX60L_Link4: geometry collision mesh filename=package://staubli/meshes/rx60l/visual/rx60bl_hb3.dae scale=0.001 0.001 0.001; visual mesh filename=package://staubli/meshes/rx60l/visual/rx60bl_hb3.dae scale=0.001 0.001 0.001
- link Staubli_RX60L_Link5: geometry collision mesh filename=package://staubli/meshes/rx60l/visual/rx60bl_hb4.dae scale=0.001 0.001 0.001; visual mesh filename=package://staubli/meshes/rx60l/visual/rx60bl_hb4.dae scale=0.001 0.001 0.001
- link Staubli_RX60L_Link6: geometry collision mesh filename=package://staubli/meshes/rx60l/visual/rx60bl_hb5.dae scale=0.001 0.001 0.001; visual mesh filename=package://staubli/meshes/rx60l/visual/rx60bl_hb5.dae scale=0.001 0.001 0.001
- link Staubli_RX60L_Link7: geometry collision mesh filename=package://staubli/meshes/rx60l/visual/rx60bl_hb6.dae scale=0.001 0.001 0.001; visual mesh filename=package://staubli/meshes/rx60l/visual/rx60bl_hb6.dae scale=0.001 0.001 0.001
