Commit message: Create RX60L xacro macro.
Also sync urdf with xacro and add xacro as run depend.

File: urdf/rx60l.urdf (robot description, URDF)
Before this commit: robot STAUBLI_RX60L, 7 links, 6 joints
Links:
- removed link Staubli_RX60L_Link1
- removed link Staubli_RX60L_Link2
- removed link Staubli_RX60L_Link3
- removed link Staubli_RX60L_Link4
- removed link Staubli_RX60L_Link5
- removed link Staubli_RX60L_Link6
- removed link Staubli_RX60L_Link7
- added link staubli_rx60l_link1; collision mesh filename=package://staubli/meshes/rx60l/visual/rx60bl_hb.dae scale=0.001 0.001 0.001; visual mesh filename=package://staubli/meshes/rx60l/visual/rx60bl_hb.dae scale=0.001 0.001 0.001
- added link staubli_rx60l_link2; collision mesh filename=package://staubli/meshes/rx60l/visual/rx60bl_hb1.dae scale=0.001 0.001 0.001; visual mesh filename=package://staubli/meshes/rx60l/visual/rx60bl_hb1.dae scale=0.001 0.001 0.001
- added link staubli_rx60l_link3; collision mesh filename=package://staubli/meshes/rx60l/visual/rx60bl_hb2.stl scale=0.001 0.001 0.001; visual mesh filename=package://staubli/meshes/rx60l/visual/rx60bl_hb2.stl scale=0.001 0.001 0.001
- added link staubli_rx60l_link4; collision mesh filename=package://staubli/meshes/rx60l/visual/rx60bl_hb3.dae scale=0.001 0.001 0.001; visual mesh filename=package://staubli/meshes/rx60l/visual/rx60bl_hb3.dae scale=0.001 0.001 0.001
- added link staubli_rx60l_link5; collision mesh filename=package://staubli/meshes/rx60l/visual/rx60bl_hb4.dae scale=0.001 0.001 0.001; visual mesh filename=package://staubli/meshes/rx60l/visual/rx60bl_hb4.dae scale=0.001 0.001 0.001
- added link staubli_rx60l_link6; collision mesh filename=package://staubli/meshes/rx60l/visual/rx60bl_hb5.dae scale=0.001 0.001 0.001; visual mesh filename=package://staubli/meshes/rx60l/visual/rx60bl_hb5.dae scale=0.001 0.001 0.001
- added link staubli_rx60l_link7; collision mesh filename=package://staubli/meshes/rx60l/visual/rx60bl_hb6.dae scale=0.001 0.001 0.001; visual mesh filename=package://staubli/meshes/rx60l/visual/rx60bl_hb6.dae scale=0.001 0.001 0.001
- added link staubli_rx60l_tool0
Joints:
- added joint joint_6-tool0: type fixed, parent staubli_rx60l_link7, child staubli_rx60l_tool0, origin xyz=0 0 0 rpy=0 0 0
- joint joint_1: child Staubli_RX60L_Link2 -> staubli_rx60l_link2; parent Staubli_RX60L_Link1 -> staubli_rx60l_link1
- joint joint_2: child Staubli_RX60L_Link3 -> staubli_rx60l_link3; parent Staubli_RX60L_Link2 -> staubli_rx60l_link2
- joint joint_3: child Staubli_RX60L_Link4 -> staubli_rx60l_link4; parent Staubli_RX60L_Link3 -> staubli_rx60l_link3
- joint joint_4: child Staubli_RX60L_Link5 -> staubli_rx60l_link5; parent Staubli_RX60L_Link4 -> staubli_rx60l_link4
- joint joint_5: child Staubli_RX60L_Link6 -> staubli_rx60l_link6; parent Staubli_RX60L_Link5 -> staubli_rx60l_link5
- joint joint_6: child Staubli_RX60L_Link7 -> staubli_rx60l_link7; parent Staubli_RX60L_Link6 -> staubli_rx60l_link6

Commit message: Add convex hull of base link STL to use as collision model.
TODO: other links.

File: urdf/rx60l.urdf (robot description, URDF)
Before this commit: robot staubli_rx60l, 8 links, 7 joints
Links:
- link staubli_rx60l_link1: geometry collision mesh filename=package://staubli/meshes/rx60l/collision/rx60bl_hb.stl scale=0.001 0.001 0.001; visual mesh filename=package://staubli/meshes/rx60l/visual/rx60bl_hb.dae scale=0.001 0.001 0.001

File: urdf/rx60l_gripper.urdf (robot description, URDF)
Before this commit: robot staubli_rx60l_gripper, 12 links, 11 joints
Links:
- link staubli_rx60l_link1: geometry collision mesh filename=package://staubli/meshes/rx60l/collision/rx60bl_hb.stl scale=0.001 0.001 0.001; visual mesh filename=package://staubli/meshes/rx60l/visual/rx60bl_hb.dae scale=0.001 0.001 0.001

File: urdf/rx60l_macro.xacro (robot description, xacro)
@@ -16,5 +16,5 @@
 				<origin xyz="0 0 0" rpy="0 0 0"/>
 				<geometry>
-					<mesh filename="package://staubli/meshes/rx60l/visual/rx60bl_hb.dae" scale="0.001 0.001 0.001"/>
+					<mesh filename="package://staubli/meshes/rx60l/collision/rx60bl_hb.stl" scale="0.001 0.001 0.001"/>
 				</geometry>
 				<material name="Blue">
